File: pcb/esp32/Temperature Control LAB ESP32.brd (EAGLE design)
At the start: 64.8 x 54.6 mm, 10 parts, among them T1 TIP31C, T2 TIP31C, U1 ESP32-DEVKIT-V1

Commit message: updates
Parts:
- moved R1 29.8 mm to (11.0, 37.5)
- moved R2 29.8 mm to (14.2, 37.5)
Connections:
- removed net 3.3V: RT1.1, RT2.1, U1.1
- removed net PIN_25: RT2.2, U1.23
- removed net PIN_26: RT1.2, U1.24
- removed net PIN_32: R2.1, U1.21
- removed net PIN_33: R1.1, U1.22
- new net PIN_12: R2.1, U1.27
- new net PIN_14: RT1.2, U1.26
- new net PIN_2: R3.2, U1.4
- new net PIN_27: RT2.2, U1.25
- new net V_LM35: RT1.1, RT2.1, U1.30
- net PIN_13: now also R1.1; no longer R3.2
Routing:
- net V_LM35: track 0.00 -> 100.5 mm
- net 3.3V: track 90.0 -> 0.00 mm
- net PIN_2: track 0.00 -> 49.1 mm
- net PIN_26: track 17.4 -> 0.00 mm
- net N$1: track 26.8 -> 12.5 mm
- net PIN_12: track 0.00 -> 14.1 mm
- net PIN_14: track 0.00 -> 12.2 mm
- net PIN_27: track 0.00 -> 9.40 mm
- net PIN_32: track 8.91 -> 0.00 mm
- net N$2: track 15.5 -> 24.2 mm
- net PIN_33: track 8.64 -> 0.00 mm
- net PIN_25: track 7.29 -> 0.00 mm
- net PIN_13: track 19.0 -> 16.1 mm
- net 5V: track 46.8 -> 46.2 mm
