File: pcb/esp32/Temperature Control LAB ESP32.sch (EAGLE design)
At the start: 10 parts, among them T1 TIP31C, T2 TIP31C, U1 ESP32-DEVKIT-V1

Commit message: updates
Connections:
- removed net 3.3V: RT1.VS+, RT2.VS+, U1.3V3
- removed net PIN_25: RT2.VOUT, U1.D25
- removed net PIN_26: RT1.VOUT, U1.D26
- removed net PIN_32: R2.1, U1.D32
- removed net PIN_33: R1.1, U1.D33
- new net PIN_12: R2.1, U1.D12
- new net PIN_14: RT1.VOUT, U1.D14
- new net PIN_2: R3.2, U1.D2
- new net PIN_27: RT2.VOUT, U1.D27
- new net V_LM35: RT1.VS+, RT2.VS+, U1.VIN
- net PIN_13: now also R1.1; no longer R3.2
Other:
- moved on the sheet: U1
Changed lines of the file:
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@@
 <part name="SUPPLY2" library="SparkFun-PowerSymbols" deviceset="5V" device=""/>
 <part name="GND3" library="SparkFun" deviceset="GND" device=""/>
-<part name="SUPPLY3" library="SparkFun-PowerSymbols" deviceset="3.3V" device=""/>
 <part name="GND4" library="SparkFun" deviceset="GND" device=""/>
-<part name="SUPPLY4" library="SparkFun-PowerSymbols" deviceset="3.3V" device=""/>
 <part name="GND5" library="SparkFun" deviceset="GND" device=""/>
 <part name="SUPPLY5" library="SparkFun-PowerSymbols" deviceset="5V" device=""/>
@@
 <part name="GND6" library="SparkFun" deviceset="GND" device=""/>
 <part name="LED1" library="led" library_urn="urn:adsk.eagle:library:259" deviceset="LED" device="5MM" package3d_urn="urn:adsk.eagle:package:15799/2"/>
-<part name="SUPPLY7" library="SparkFun-PowerSymbols" deviceset="3.3V" device=""/>
 <part name="GND7" library="SparkFun" deviceset="GND" device=""/>
 <part name="RT1" library="TMP36GT9Z" deviceset="TMP36GT9Z" device=""/>
@@
 <attribute name="VALUE" x="20.32" y="43.18" size="1.778" layer="96"/>
 </instance>
-<instance part="SUPPLY3" gate="G$1" x="20.32" y="63.5" smashed="yes">
-<attribute name="VALUE" x="20.32" y="66.294" size="1.778" layer="96" align="bottom-center"/>
-</instance>
 <instance part="GND4" gate="1" x="55.88" y="45.72" smashed="yes">
 <attribute name="VALUE" x="53.34" y="43.18" size="1.778" layer="96"/>
-</instance>
-<instance part="SUPPLY4" gate="G$1" x="53.34" y="63.5" smashed="yes">
-<attribute name="VALUE" x="53.34" y="66.294" size="1.778" layer="96" align="bottom-center"/>
 </instance>
 <instance part="GND5" gate="1" x="-78.74" y="17.78" smashed="yes">
@@
 <attribute name="VALUE" x="98.552" y="66.675" size="1.778" layer="96" rot="R180"/>
 </instance>
-<instance part="SUPPLY7" gate="G$1" x="-35.56" y="22.86" smashed="yes">
-<attribute name="VALUE" x="-35.56" y="25.654" size="1.778" layer="96" align="bottom-center"/>
-</instance>
-<instance part="GND7" gate="1" x="-38.1" y="-40.64" smashed="yes">
-<attribute name="VALUE" x="-40.64" y="-43.18" size="1.778" layer="96"/>
+<instance part="GND7" gate="1" x="-27.94" y="-40.64" smashed="yes">
+<attribute name="VALUE" x="-30.48" y="-43.18" size="1.778" layer="96"/>
 </instance>
 <instance part="RT1" gate="G$1" x="20.32" y="55.88" smashed="yes" rot="R180">
@@
 <attribute name="VALUE" x="34.29" y="50.8" size="1.778" layer="96" rot="R180" align="center-left"/>
 </instance>
-<instance part="U1" gate="G$1" x="-55.88" y="-10.16" smashed="yes">
-<attribute name="VALUE" x="-66.04" y="-40.64" size="1.778" layer="96"/>
-<attribute name="NAME" x="-66.04" y="20.32" size="1.778" layer="95" align="top-left"/>
+<instance part="U1" gate="G$1" x="-45.72" y="-10.16" smashed="yes">
+<attribute name="VALUE" x="-55.88" y="-40.64" size="1.778" layer="96"/>
+<attribute name="NAME" x="-55.88" y="20.32" size="1.778" layer="95" align="top-left"/>
 </instance>
 </instances>
@@
 <segment>
 <pinref part="GND7" gate="1" pin="GND"/>
-<wire x1="-38.1" y1="-38.1" x2="-38.1" y2="-35.56" width="0.1524" layer="91"/>
+<wire x1="-27.94" y1="-38.1" x2="-27.94" y2="-35.56" width="0.1524" layer="91"/>
 <pinref part="U1" gate="G$1" pin="GND"/>
-<wire x1="-38.1" y1="-35.56" x2="-40.64" y2="-35.56" width="0.1524" layer="91"/>
+<wire x1="-27.94" y1="-35.56" x2="-30.48" y2="-35.56" width="0.1524" layer="91"/>
 </segment>
 </net>
@@
 </segment>
 </net>
-<net name="3.3V" class="0">
-<segment>
-<pinref part="SUPPLY3" gate="G$1" pin="3.3V"/>
-<wire x1="20.32" y1="60.96" x2="20.32" y2="63.5" width="0.1524" layer="91"/>
-<pinref part="RT1" gate="G$1" pin="VS+"/>
-</segment>
-<segment>
-<pinref part="SUPPLY4" gate="G$1" pin="3.3V"/>
-<wire x1="53.34" y1="60.96" x2="53.34" y2="63.5" width="0.1524" layer="91"/>
-<pinref part="RT2" gate="G$1" pin="VS+"/>
-</segment>
-<segment>
-<pinref part="SUPPLY7" gate="G$1" pin="3.3V"/>
-<wire x1="-35.56" y1="15.24" x2="-35.56" y2="22.86" width="0.1524" layer="91"/>
-<pinref part="U1" gate="G$1" pin="3V3"/>
-<wire x1="-40.64" y1="15.24" x2="-35.56" y2="15.24" width="0.1524" layer="91"/>
-</segment>
-</net>
 <net name="N$3" class="0">
 <segment>
@@
 </segment>
 </net>
-<net name="PIN_25" class="0">
-<segment>
-<wire x1="-40.64" y1="-12.7" x2="-38.1" y2="-12.7" width="0.1524" layer="91"/>
-<label x="-38.1" y="-12.7" size="1.016" layer="95" xref="yes"/>
-<pinref part="U1" gate="G$1" pin="D25"/>
-</segment>
-<segment>
-<wire x1="53.34" y1="58.42" x2="55.88" y2="58.42" width="0.1524" layer="91"/>
-<label x="55.88" y="58.42" size="1.016" layer="95" xref="yes"/>
-<pinref part="RT2" gate="G$1" pin="VOUT"/>
-</segment>
-</net>
-<net name="PIN_26" class="0">
-<segment>
-<wire x1="-40.64" y1="-15.24" x2="-38.1" y2="-15.24" width="0.1524" layer="91"/>
-<label x="-38.1" y="-15.24" size="1.016" layer="95" xref="yes"/>
-<pinref part="U1" gate="G$1" pin="D26"/>
-</segment>
+<net name="PIN_13" class="0">
+<segment>
+<wire x1="-60.96" y1="-17.78" x2="-63.5" y2="-17.78" width="0.1524" layer="91"/>
+<label x="-63.5" y="-17.78" size="1.016" layer="95" rot="R180" xref="yes"/>
+<pinref part="U1" gate="G$1" pin="D13"/>
+</segment>
+<segment>
+<pinref part="R1" gate="G$1" pin="1"/>
+<wire x1="-60.96" y1="58.42" x2="-63.5" y2="58.42" width="0.1524" layer="91"/>
+<label x="-63.5" y="58.42" size="1.016" layer="95" rot="R180" xref="yes"/>
+</segment>
+</net>
+<net name="PIN_12" class="0">
+<segment>
+<wire x1="-60.96" y1="-15.24" x2="-63.5" y2="-15.24" width="0.1524" layer="91"/>
+<label x="-63.5" y="-15.24" size="1.016" layer="95" rot="R180" xref="yes"/>
+<pinref part="U1" gate="G$1" pin="D12"/>
+</segment>
+<segment>
+<pinref part="R2" gate="G$1" pin="1"/>
+<wire x1="-33.02" y1="58.42" x2="-35.56" y2="58.42" width="0.1524" layer="91"/>
+<label x="-35.56" y="58.42" size="1.016" layer="95" rot="R180" xref="yes"/>
+</segment>
+</net>
+<net name="PIN_14" class="0">
 <segment>
 <wire x1="20.32" y1="58.42" x2="22.86" y2="58.42" width="0.1524" layer="91"/>
@@
 <label x="22.86" y="58.42" size="1.016" layer="95" xref="yes"/>
 </segment>
-</net>
-<net name="PIN_32" class="0">
-<segment>
-<wire x1="-40.64" y1="-20.32" x2="-38.1" y2="-20.32" width="0.1524" layer="91"/>
-<label x="-38.1" y="-20.32" size="1.016" layer="95" xref="yes"/>
-<pinref part="U1" gate="G$1" pin="D32"/>
-</segment>
-<segment>
-<pinref part="R2" gate="G$1" pin="1"/>
-<wire x1="-33.02" y1="58.42" x2="-35.56" y2="58.42" width="0.1524" layer="91"/>
-<label x="-35.56" y="58.42" size="1.016" layer="95" rot="R180" xref="yes"/>
-</segment>
-</net>
-<net name="PIN_33" class="0">
-<segment>
-<wire x1="-40.64" y1="-22.86" x2="-38.1" y2="-22.86" width="0.1524" layer="91"/>
-<label x="-38.1" y="-22.86" size="1.016" layer="95" xref="yes"/>
-<pinref part="U1" gate="G$1" pin="D33"/>
-</segment>
-<segment>
-<pinref part="R1" gate="G$1" pin="1"/>
-<wire x1="-60.96" y1="58.42" x2="-63.5" y2="58.42" width="0.1524" layer="91"/>
-<label x="-63.5" y="58.42" size="1.016" layer="95" rot="R180" xref="yes"/>
-</segment>
-</net>
-<net name="PIN_13" class="0">
+<segment>
+<wire x1="-60.96" y1="-20.32" x2="-63.5" y2="-20.32" width="0.1524" layer="91"/>
+<label x="-63.5" y="-20.32" size="1.016" layer="95" rot="R180" xref="yes"/>
+<pinref part="U1" gate="G$1" pin="D14"/>
+</segment>
+</net>
+<net name="PIN_27" class="0">
+<segment>
+<wire x1="53.34" y1="58.42" x2="55.88" y2="58.42" width="0.1524" layer="91"/>
+<label x="55.88" y="58.42" size="1.016" layer="95" xref="yes"/>
+<pinref part="RT2" gate="G$1" pin="VOUT"/>
+</segment>
+<segment>
+<wire x1="-30.48" y1="-17.78" x2="-27.94" y2="-17.78" width="0.1524" layer="91"/>
+<label x="-27.94" y="-17.78" size="1.016" layer="95" xref="yes"/>
+<pinref part="U1" gate="G$1" pin="D27"/>
+</segment>
+</net>
+<net name="PIN_2" class="0">
 <segment>
 <pinref part="R3" gate="G$1" pin="2"/>
@@
 </segment>
 <segment>
-<wire x1="-71.12" y1="-17.78" x2="-73.66" y2="-17.78" width="0.1524" layer="91"/>
-<label x="-73.66" y="-17.78" size="1.016" layer="95" rot="R180" xref="yes"/>
-<pinref part="U1" gate="G$1" pin="D13"/>
-</segment>
-</net>
+<wire x1="-60.96" y1="-7.62" x2="-63.5" y2="-7.62" width="0.1524" layer="91"/>
+<label x="-63.5" y="-7.62" size="1.016" layer="95" rot="R180" xref="yes"/>
+<pinref part="U1" gate="G$1" pin="D2"/>
+</segment>
+</net>
+<net name="V_LM35" class="0">
+<segment>
+<pinref part="RT1" gate="G$1" pin="VS+"/>
+<wire x1="20.32" y1="60.96" x2="22.86" y2="60.96" width="0.1524" layer="91"/>
+<label x="22.86" y="60.96" size="1.016" layer="95" xref="yes"/>
+</segment>
+<segment>
+<pinref part="RT2" gate="G$1" pin="VS+"/>
+<wire x1="53.34" y1="60.96" x2="55.88" y2="60.96" width="0.1524" layer="91"/>
+<label x="55.88" y="60.96" size="1.016" layer="95" xref="yes"/>
+</segment>
+<segment>
+<pinref part="U1" gate="G$1" pin="VIN"/>
+<wire x1="-60.96" y1="15.24" x2="-63.5" y2="15.24" width="0.1524" layer="91"/>
+<label x="-63.5" y="15.24" size="1.016" layer="95" rot="R180" xref="yes"/>
+</segment>
+</net>
